File: 1U VCA.kicad_pcb (KiCad board)
At the start: 2 copper layers, 27.9 x 28.7 mm, 8 parts, among them J1 IN1, J2 CV1, J3 OUT1, J4 IN2, J5 CV2, J6 OUT2

Commit message: Not sure what was changed, but this is still not the final design
Parts:
- removed LED1, LED2: LED, LEDs:LED_D3.0mm_FlatTop
- added C1: 100n, Capacitor_SMD:C_0603_1608Metric_Pad1.05x0.95mm_HandSolder, F.Cu at (93.8, 39.1)
- added C2: 100n, Capacitor_SMD:C_0603_1608Metric_Pad1.05x0.95mm_HandSolder, F.Cu at (101.9, 31.7)
- added C3: 100n, Capacitor_SMD:C_0603_1608Metric_Pad1.05x0.95mm_HandSolder, F.Cu at (87.6, 45.7)
- added C4: 100n, Capacitor_SMD:C_0603_1608Metric_Pad1.05x0.95mm_HandSolder, F.Cu at (80.9, 45.5)
- added C5: 100n, Capacitor_SMD:C_0603_1608Metric_Pad1.05x0.95mm_HandSolder, F.Cu at (97.1, 34.8)
- added C6: 100n, Capacitor_SMD:C_0603_1608Metric_Pad1.05x0.95mm_HandSolder, F.Cu at (101.9, 30.2)
- added C7: 10u, Capacitor_SMD:CP_Elec_4x5.4, F.Cu at (80.4, 25.8)
- added C8: 10u, Capacitor_SMD:CP_Elec_4x5.4, F.Cu at (80.7, 30.8)
- added D1: 1N4148, Diode_SMD:D_0603_1608Metric_Pad1.05x0.95mm_HandSolder, F.Cu at (87.3, 50.5)
- added D2: 1N4148, Diode_SMD:D_0603_1608Metric_Pad1.05x0.95mm_HandSolder, F.Cu at (77.5, 37.8)
- added J7: OUT2, KraakenStuff:PJ301M-12, B.Cu at (45.7, 66.1)
- added JP1: Jumper, Connector_PinHeader_2.54mm:PinHeader_1x02_P2.54mm_Vertical, F.Cu at (98.4, 29.7)
- added JP2: Jumper, Connector_PinHeader_2.54mm:PinHeader_1x02_P2.54mm_Vertical, F.Cu at (84.4, 40.4)
- added Q1: MMBT3906, Package_TO_SOT_SMD:SOT-23, F.Cu at (91.4, 50.2)
- added Q2: MMBT3906, Package_TO_SOT_SMD:SOT-23, F.Cu at (109.1, 51.1)
- added R1: 1M, Resistor_SMD:R_0603_1608Metric_Pad1.05x0.95mm_HandSolder, F.Cu at (87.9, 42.6)
- added R10: 1M, Resistor_SMD:R_0603_1608Metric_Pad1.05x0.95mm_HandSolder, F.Cu at (91.0, 45.7)
- added R11: 390R, Resistor_SMD:R_0603_1608Metric_Pad1.05x0.95mm_HandSolder, F.Cu at (97.1, 39.3)
- added R12: 15k, Resistor_SMD:R_0603_1608Metric_Pad1.05x0.95mm_HandSolder, F.Cu at (94.6, 42.1)
- added R13: 100k, Resistor_SMD:R_0603_1608Metric_Pad1.05x0.95mm_HandSolder, F.Cu at (97.1, 37.8)
- added R14: 390R, Resistor_SMD:R_0603_1608Metric_Pad1.05x0.95mm_HandSolder, F.Cu at (87.9, 44.2)
- added R15: 20k, Resistor_SMD:R_0603_1608Metric_Pad1.05x0.95mm_HandSolder, F.Cu at (93.8, 40.6)
- added R16: 20k, Resistor_SMD:R_0603_1608Metric_Pad1.05x0.95mm_HandSolder, F.Cu at (101.9, 33.2)
- added R17: 39k, Resistor_SMD:R_0603_1608Metric_Pad1.05x0.95mm_HandSolder, F.Cu at (100.4, 34.8)
- added R18: 300k, Resistor_SMD:R_0603_1608Metric_Pad1.05x0.95mm_HandSolder, F.Cu at (97.1, 36.3)
- added R2: 390R, Resistor_SMD:R_0603_1608Metric_Pad1.05x0.95mm_HandSolder, F.Cu at (91.2, 42.6)
- added R3: 15k, Resistor_SMD:R_0603_1608Metric_Pad1.05x0.95mm_HandSolder, F.Cu at (84.3, 45.5)
- added R4: 100k, Resistor_SMD:R_0603_1608Metric_Pad1.05x0.95mm_HandSolder, F.Cu at (91.2, 44.2)
- added R5: 390R, Resistor_SMD:R_0603_1608Metric_Pad1.05x0.95mm_HandSolder, F.Cu at (100.5, 39.3)
- added R6: 20k, Resistor_SMD:R_0603_1608Metric_Pad1.05x0.95mm_HandSolder, F.Cu at (97.9, 40.8)
- added R7: 20k, Resistor_SMD:R_0603_1608Metric_Pad1.05x0.95mm_HandSolder, F.Cu at (100.5, 37.8)
- added R8: 39k, Resistor_SMD:R_0603_1608Metric_Pad1.05x0.95mm_HandSolder, F.Cu at (94.6, 43.6)
- added R9: 300k, Resistor_SMD:R_0603_1608Metric_Pad1.05x0.95mm_HandSolder, F.Cu at (100.4, 36.3)
- added RV1: 100k, Potentiometer_THT:Potentiometer_Bourns_3266Y_Vertical, F.Cu at (52.6, 47.5)
- added RV2: 100k, Potentiometer_THT:Potentiometer_Bourns_3266Y_Vertical, F.Cu at (52.6, 58.7)
- added U1: TL074, Package_SO:TSSOP-14_4.4x5mm_P0.65mm, F.Cu at (99.3, 50.1)
- added U2: LM13700, Package_SO:SOIC-16_3.9x9.9mm_P1.27mm, F.Cu at (99.5, 60.2)
- J1, J2, J3, J5: footprint 4ms-footprints:PJ301M-12 -> KraakenStuff:PJ301M-12; moved to B.Cu
- J4: value IN2 -> Conn_01x03; footprint 4ms-footprints:PJ301M-12 -> Connector_PinHeader_2.54mm:PinHeader_1x03_P2.54mm_Vertical
- J6: value OUT2 -> IN2; footprint 4ms-footprints:PJ301M-12 -> KraakenStuff:PJ301M-12; moved to B.Cu
- moved J4 57.3 mm to (116.4, 35.5)
- moved J1 22.7 mm to (59.7, 45.2), turned to 180 degrees
- moved J2 22.7 mm to (59.7, 55.6), turned to 180 degrees
- moved J5 22.7 mm to (45.7, 55.7), turned to 0 degrees
- moved J3 22.7 mm to (59.7, 66.1), turned to 180 degrees
- moved J6 14.3 mm to (45.7, 45.2), turned to 0 degrees
Connections:
- J4 pad 1: Net-(J4-Pad1) -> +12V
- J4 pad 2: Net-(J4-Pad2) -> GND
- J4 pad 3: Net-(J4-Pad3) -> -12V
